File: hardware/esproomba.kicad_pcb (KiCad board)
At the start: 2 copper layers, 20 x 51.5 mm, 16 parts, among them J1 CONN-7, J2 CONN-5, M1 ESP-12, M2 V-REG, U1 MMA8652FC

Commit message: v0.2
Parts:
- removed C4: 0.1uF, SMD-1608:SMD-1608
- added R6: 4.7k, SMD-1608:SMD-1608, F.Cu at (161.7, 103.7)
- D1: value D -> LED; footprint libs:SOD-523 -> libs:SMD-1608-LED
- D2: value LED -> D; footprint libs:SMD-1608-LED -> libs:SOD-523
- J2: value CONN-5 -> CONN-6; footprint libs:CONN-5-0.1 -> libs:CONN-6
- R4: value 1k -> 4.7k
- U1: footprint DFN-10:DFN-10 -> libs:DFN-10
- moved C3 43.1 mm to (154.7, 101.1), turned to 270 degrees
- moved R1 42.4 mm to (158.3, 103.7)
- moved C1 40.0 mm to (160.0, 103.7)
- moved D2 39.7 mm to (166.7, 102.7)
- moved D1 39.3 mm to (163.4, 102.8), turned to 180 degrees
- moved R4 38.2 mm to (160.9, 101.1), turned to 270 degrees
- moved R3 37.9 mm to (165.1, 102.8), turned to 180 degrees
- moved R2 37.6 mm to (151.2, 102.8)
- moved U1 36.7 mm to (154.7, 103.3), turned to 180 degrees
- moved J1 36.3 mm to (158.5, 126.5)
- moved M1 36.3 mm to (158.5, 83.3)
- moved M2 35.9 mm to (158.4, 116.2)
- moved C2 34.5 mm to (154.7, 105.5), turned to 270 degrees
- moved J2 30.6 mm to (160.2, 107.9)
- moved R5 30.5 mm to (151.2, 107.1), turned to 0 degrees
Connections:
- D1 pad C: /TX -> Net-(D1-PadC)
- D2 pad C: DGND -> /TX
- J1 pad 5: /DD -> (no net)
- J2 pad 1: /RX -> DGND
- J2 pad 2: /TX -> /BATT
- J2 pad 3: /GPIO0 -> /TX
- J2 pad 4: /CH_PD -> /RX
- J2 pad 5: DGND -> /GPIO0
- M1 pad 1: +3V3 -> /WAKE
- M1 pad 10: Net-(M1-Pad10) -> DGND
- M1 pad 11: Net-(M1-Pad11) -> Net-(D1-PadC)
- M1 pad 14: /SDA -> (no net)
- M1 pad 15: Net-(D1-PadA) -> Net-(D2-PadA)
- M1 pad 2: Net-(M1-Pad2) -> (no net)
- M1 pad 4: +3V3 -> /WAKE
- M1 pad 5: /INT1 -> /INT2
- M1 pad 6: /INT2 -> /INT1
- M1 pad 7: /DD -> /SDA
- R3 pad 1: Net-(M1-Pad10) -> +3V3
- R3 pad 2: DGND -> Net-(D2-PadA)
- R4 pad 1: Net-(M1-Pad11) -> +3V3
- R4 pad 2: Net-(D2-PadA) -> /WAKE
- R5 pad 2: Net-(D1-PadA) -> /CH_PD
- U1 pad 3: /INT1 -> /INT2
- U1 pad 5: /INT2 -> /INT1
Routing:
- net /DD: track 38.7 -> 0.00 mm
- net /WAKE: track 0.00 -> 26.0 mm
- net Net-(D1-PadA): track 25.2 -> 2.07 mm, vias 2 -> 0
- net Net-(D2-PadA): track 2.17 -> 20.6 mm
- net /SDA: track 27.4 -> 12.0 mm
- net +3V3: track 58.5 -> 44.2 mm
- net Net-(M1-Pad11): track 13.8 -> 0.00 mm
- net Net-(M1-Pad10): track 12.4 -> 0.00 mm
- net Net-(D1-PadC): track 0.00 -> 10.4 mm
- net /GPIO0: track 12.8 -> 21.1 mm, vias 0 -> 1
- net /CH_PD: track 18.2 -> 24.9 mm, vias 0 -> 1
- net /INT2: track 9.80 -> 15.9 mm
- net /TX: track 30.7 -> 25.8 mm, vias 0 -> 2
- net /SCL: track 24.4 -> 20.2 mm
- net DGND: track 15.7 -> 19.8 mm
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Other:
- board size 20 x 51.5 mm -> 20 x 50.5 mm
- board text added: "esproomba v0.2"
- board text removed: "esproomba 0.1v"
