File: hardware/esproomba.sch (KiCad schematic (older format))
At the start: 16 parts, among them J1 CONN-7, J2 CONN-5, M1 ESP-12, M2 V-REG, U1 MMA8652FC

Commit message: v0.2
Parts:
- removed C4: 0.1uF, SMD-1608:SMD-1608, symbol C
- removed D2: LED, libs:SMD-1608-LED, symbol LED
- removed J2: CONN-5, libs:CONN-5-0.1, symbol CONN-5
- removed R3: 4.7k, SMD-1608:SMD-1608, symbol R
- added D1: LED, libs:SMD-1608-LED, symbol LED
- added J2: CONN-6, libs:CONN-6, symbol CONN-6
- added R5, R6: 4.7k, SMD-1608:SMD-1608, symbol R
- R4: value 1k -> 4.7k
- U1: footprint DFN-10:DFN-10 -> libs:DFN-10
- renumbered D1 to D2, R5 to R3
Connections:
- net +3V3: now also R4.1, R5.1, R6.1; no longer M1.1 (~RST), M1.4 (GPIO16/~WAKE)
- net BATT: now also J2.2
- net CH_PD: now also J2.6, R5.2
- net DGND: now also M1.10 (MTDO/GPIO15), J2.1
- net GPIO0: now also J2.5
- net INT1: now also M1.6 (GPIO12), U1.5 (INT2); no longer M1.5 (GPIO14), U1.3 (INT1)
- net INT2: now also M1.5 (GPIO14), U1.3 (INT1); no longer M1.6 (GPIO12), U1.5 (INT2)
- net RX: now also J2.4
- net SDA: now also M1.7 (GPIO13); no longer M1.14 (GPIO4)
- net TX: now also J2.3
- net at M1.11 (GPIO2): now also D1.C; no longer R4.1
- net WAKE: now reaches R4.2
- net WAKE: now also M1.1 (~RST), M1.4 (GPIO16/~WAKE)
- net DD: no longer names the net of J1.5
- net DD: no longer M1.7 (GPIO13)
- new net: D1.A, R6.2
- no-connect marks 1 -> 3
Other:
- moved on the sheet: D2, J1, M1, M2, R3
